File: ch573beacon.kicad_sch (KiCad schematic)
At the start: 32 parts, among them U1 BH1750FVI

Commit message: update
Parts:
- added C11: 2.2uf, Capacitor_SMD:C_0402_1005Metric, symbol Device:C
- AE1: value (none) -> Antenna; footprint (none) -> my:CA-C03
- BT1: value (none) -> Battery; footprint (none) -> Battery:BatteryHolder_Keystone_1058_1x2032
- C1, C2: value (none) -> 2.2uf; footprint (none) -> Capacitor_SMD:C_0402_1005Metric
- C10: value (none) -> 10uf
- C5, C6, C9: value (none) -> 0.1uf; footprint (none) -> Capacitor_SMD:C_0402_1005Metric
- C8: value (none) -> 4.7uf
- D1: value (none) -> LED; footprint (none) -> LED_SMD:LED_0402_1005Metric
- J1: value (none) -> USB_C_Receptacle_USB2.0; footprint (none) -> Connector_USB:USB_C_Receptacle_HRO_TYPE-C-31-M-12
- L1: value (none) -> 22uh; footprint (none) -> Inductor_SMD:L_Taiyo-Yuden_MD-2020
- R1, R2: value (none) -> 4.7k; footprint (none) -> Resistor_SMD:R_0402_1005Metric
- R3: value (none) -> 1k; footprint (none) -> Resistor_SMD:R_0402_1005Metric
- R4, R5: value (none) -> 10k; footprint (none) -> Resistor_SMD:R_0402_1005Metric
- R6: value (none) -> 5.1k; footprint (none) -> Resistor_SMD:R_0402_1005Metric
- R8: value (none) -> 2k; footprint (none) -> Resistor_SMD:R_0402_1005Metric
- R9: value (none) -> 1k
- SW1: value (none) -> SW_Push; footprint (none) -> my:bt-342
- U2: value (none) -> ME6216A33M3G; footprint (none) -> Package_TO_SOT_SMD:SOT-23
- U3: value (none) -> CH573F; footprint (none) -> Package_DFN_QFN:QFN-28-1EP_4x4mm_P0.45mm_EP2.4x2.4mm
- U4: value (none) -> SHT31-DIS; footprint (none) -> Sensor_Humidity:Sensirion_DFN-8-1EP_2.5x2.5mm_P0.5mm_EP1.1x1.7mm
- U5: value (none) -> TP4054; footprint (none) -> Package_TO_SOT_SMD:SOT-23-5
- Y1: value (none) -> Crystal; footprint (none) -> Crystal:Crystal_SMD_2012-2Pin_2.0x1.2mm_HandSoldering
- Y2: value (none) -> Crystal_GND24; footprint (none) -> Crystal:Crystal_SMD_2016-4Pin_2.0x1.6mm
Connections:
- net SCL is gone; now on net SCL_BH: R1.2, U1.6 (SCL)
- net SDA is gone; now on net SDA_BH: R2.2, U1.4 (SDA)
- net GND: now also C11.1
- net SCL_SHT: now also U3.7 (PA9)
- net SDA_SHT: now also U3.6 (PA8)
- net VCC: now also C2.2, U3.5 (VIO33)
- net at U3.20 (VINTA): now also C11.2
- net SCL_BH: now reaches U3.8 (PB15)
- net SDA_BH: now reaches U3.9 (PB14)
- no-connect marks 5 -> 4
Other:
- moved on the sheet: C2

Commit message: update
Parts:
- removed AE1: Antenna, my:CA-C03, symbol Device:Antenna
- added AE1: (no value), symbol Device:Antenna_Chip
- added D1: (no value), symbol Device:D
- added H1: (no value), symbol Mechanical:MountingHole
- added H2: MountingHole, MountingHole:MountingHole_2.2mm_M2, symbol Mechanical:MountingHole
- added JP1: (no value), symbol Jumper:Jumper_3_Bridged12
- renumbered C9 to C10, C10 to C11, C11 to C7, C7 to C8, C8 to C9, D1 to D2
Connections:
- net +3V3 is gone; now on net VCC: R1.1, R2.1, R3.1, U1.1 (VCC)
- net +5V: now also JP1.2 (C); no longer C9.1, R9.1, U5.4 (VDD)
- net BAT: now also D1.2 (A); no longer C3.1, U2.3 (VIN)
- net SCL_BH: now also U3.6 (PA8); no longer U3.8 (PB15)
- net SCL_SHT: now also U3.8 (PB15); no longer U3.7 (PA9)
- net SDA_BH: now also U3.7 (PA9); no longer U3.9 (PB14)
- net SDA_SHT: now also U3.9 (PB14); no longer U3.6 (PA8)
- net at U3.21 (ANT): now also AE1.2 (PCB_Trace)
- new net CHARG: C9.1, JP1.3 (B), R9.1, U5.4 (VDD)
- new net DIRECT: C3.1, D1.1 (K), JP1.1 (A), U2.3 (VIN)
- no-connect marks 4 -> 13

Commit message: update
Parts:
- removed H1: (no value), symbol Mechanical:MountingHole
- removed H2: MountingHole, MountingHole:MountingHole_2.2mm_M2, symbol Mechanical:MountingHole
- AE1: value (none) -> Antenna_Chip; footprint (none) -> BLab:CA-03
- C3, C4: value 4.7uf -> (none)
- D1: value (none) -> D; footprint (none) -> Diode_SMD:D_0402_1005Metric
- JP1: value (none) -> Jumper_3_Bridged12; footprint (none) -> Jumper:SolderJumper-3_P1.3mm_Open_RoundedPad1.0x1.5mm
Changed lines of the file:
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@@
     (in_bom yes) (on_board yes) (fields_autoplaced)
     (property "Reference" "JP1" (id 0) (at 179.07 133.35 0))
-    (property "Value" "" (id 1) (at 179.07 135.89 0))
-    (property "Footprint" "" (id 2) (at 179.07 139.7 0)
+    (property "Value" "Jumper_3_Bridged12" (id 1) (at 179.07 135.89 0))
+    (property "Footprint" "Jumper:SolderJumper-3_P1.3mm_Open_RoundedPad1.0x1.5mm" (id 2) (at 179.07 139.7 0)
       (effects (font (size 1.27 1.27)) hide)
     )
@@
     (pin "1")
     (pin "2")
-  )
-  (symbol (lib_id "Mechanical:MountingHole") (at 116.84 106.68 0) (unit 1)
-    (in_bom yes) (on_board yes) (fields_autoplaced)
-    (property "Reference" "H1" (id 0) (at 119.38 105.4099 0)
-      (effects (font (size 1.27 1.27)) (justify left))
-    )
-    (property "Value" "" (id 1) (at 119.38 107.9499 0)
-      (effects (font (size 1.27 1.27)) (justify left))
-    )
-    (property "Footprint" "" (id 2) (at 116.84 106.68 0)
-      (effects (font (size 1.27 1.27)) hide)
-    )
-    (property "Datasheet" "~" (id 3) (at 116.84 106.68 0)
-      (effects (font (size 1.27 1.27)) hide)
-    )
   )
   (symbol (lib_id "Device:R") (at 237.49 146.05 0) (unit 1)
@@
     (in_bom yes) (on_board yes) (fields_autoplaced)
     (property "Reference" "D1" (id 0) (at 45.72 106.68 0))
-    (property "Value" "" (id 1) (at 45.72 109.22 0))
-    (property "Footprint" "" (id 2) (at 45.72 113.03 0)
+    (property "Value" "D" (id 1) (at 45.72 109.22 0))
+    (property "Footprint" "Diode_SMD:D_0402_1005Metric" (id 2) (at 45.72 113.03 0)
       (effects (font (size 1.27 1.27)) hide)
     )
@@
     (pin "2")
   )
-  (symbol (lib_id "Mechanical:MountingHole") (at 116.84 114.3 0) (unit 1)
-    (in_bom yes) (on_board yes) (fields_autoplaced)
-    (property "Reference" "H2" (id 0) (at 119.38 113.0299 0)
-      (effects (font (size 1.27 1.27)) (justify left))
-    )
-    (property "Value" "MountingHole" (id 1) (at 119.38 115.5699 0)
-      (effects (font (size 1.27 1.27)) (justify left))
-    )
-    (property "Footprint" "MountingHole:MountingHole_2.2mm_M2" (id 2) (at 116.84 114.3 0)
-      (effects (font (size 1.27 1.27)) hide)
-    )
-    (property "Datasheet" "~" (id 3) (at 116.84 114.3 0)
-      (effects (font (size 1.27 1.27)) hide)
-    )
-  )
   (symbol (lib_id "power:GND") (at 78.74 35.56 180) (unit 1)
     (in_bom yes) (on_board yes) (fields_autoplaced)
@@
       (effects (font (size 1.27 1.27)) (justify left))
     )
-    (property "Value" "" (id 1) (at 104.14 38.0999 0)
-      (effects (font (size 1.27 1.27)) (justify left))
-    )
-    (property "Footprint" "" (id 2) (at 96.52 34.925 0)
+    (property "Value" "Antenna_Chip" (id 1) (at 104.14 38.0999 0)
+      (effects (font (size 1.27 1.27)) (justify left))
+    )
+    (property "Footprint" "BLab:CA-03" (id 2) (at 96.52 34.925 0)
       (effects (font (size 1.27 1.27)) hide)
     )
@@
       (effects (font (size 1.27 1.27)) (justify right))
     )
-    (property "Value" "0.1uf" (id 1) (at 243.84 49.53 90)
+    (property "Value" "0.1uf" (id 1) (at 248.92 48.26 90)
       (effects (font (size 1.27 1.27)) (justify right))
     )
@@
       (effects (font (size 1.27 1.27)) (justify right))
     )
-    (property "Value" "4.7uf" (id 1) (at 45.72 114.3 90)
+    (property "Value" "" (id 1) (at 45.72 114.3 90)
       (effects (font (size 1.27 1.27)) (justify right))
     )
@@
       (effects (font (size 1.27 1.27)) (justify right))
     )
-    (property "Value" "4.7uf" (id 1) (at 72.39 114.3 90)
+    (property "Value" "" (id 1) (at 72.39 114.3 90)
       (effects (font (size 1.27 1.27)) (justify right))
     )
@@
     )
     (path "/c0c5f40e-b48e-484e-b7d5-f853094e389e"
-      (reference "C3") (unit 1) (value "4.7uf") (footprint "Capacitor_SMD:C_0402_1005Metric")
+      (reference "C3") (unit 1) (value "0.1uf") (footprint "Capacitor_SMD:C_0402_1005Metric")
     )
     (path "/e5ea9f01-f000-4b9e-a7e4-ff7067319780"
-      (reference "C4") (unit 1) (value "4.7uf") (footprint "Capacitor_SMD:C_0402_1005Metric")
+      (reference "C4") (unit 1) (value "0.1uf") (footprint "Capacitor_SMD:C_0402_1005Metric")
     )
     (path "/38bb4d15-6633-42cb-a1f7-5428d09f7029"
@@
       (reference "D2") (unit 1) (value "LED") (footprint "LED_SMD:LED_0402_1005Metric")
     )
-    (path "/5ed581cd-7566-4d2e-92de-125e9c99efd5"
-      (reference "H1") (unit 1) (value "MountingHole") (footprint "MountingHole:MountingHole_2.2mm_M2")
-    )
-    (path "/a5931523-7d56-4ec0-a4e5-f1fa1da7fa52"
-      (reference "H2") (unit 1) (value "MountingHole") (footprint "MountingHole:MountingHole_2.2mm_M2")
-    )
     (path "/9c9e0f77-bda3-41a8-8ee4-7f92da443b6d"

Commit message: update
Parts:
- C3, C4: value (none) -> 0.1uf
- C9: value 4.7uf -> (none)
Other:
- note added: "当电池充满以后指示灯亮 2k 电流360ma"
- note removed: "当电池充满以后指示灯亮"
Changed lines of the file:
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@@
     (effects (font (size 1.27 1.27)) (justify left bottom))
   )
-  (text "当电池充满以后指示灯亮" (at 224.79 160.02 0)
+  (text "当电池充满以后指示灯亮  2k 电流360ma" (at 228.6 161.29 0)
     (effects (font (size 1.27 1.27)) (justify left bottom))
   )
@@
       (effects (font (size 1.27 1.27)) (justify right))
     )
-    (property "Value" "" (id 1) (at 45.72 114.3 90)
+    (property "Value" "0.1uf" (id 1) (at 45.72 114.3 90)
       (effects (font (size 1.27 1.27)) (justify right))
     )
@@
       (effects (font (size 1.27 1.27)) (justify right))
     )
-    (property "Value" "4.7uf" (id 1) (at 242.57 123.19 90)
+    (property "Value" "" (id 1) (at 242.57 123.19 90)
       (effects (font (size 1.27 1.27)) (justify right))
     )
@@
       (effects (font (size 1.27 1.27)) (justify right))
     )
-    (property "Value" "" (id 1) (at 72.39 114.3 90)
+    (property "Value" "0.1uf" (id 1) (at 72.39 114.3 90)
       (effects (font (size 1.27 1.27)) (justify right))
     )
@@
     )
     (path "/e30a3608-08cd-4a62-83ba-3c7b7128658a"
-      (reference "C9") (unit 1) (value "4.7uf") (footprint "Capacitor_SMD:C_0402_1005Metric")
+      (reference "C9") (unit 1) (value "1uf") (footprint "Capacitor_SMD:C_0402_1005Metric")
     )
     (path "/b87cc950-20d9-41d8-a76f-ab1ab7740cb0"
